File: experiments/schematics/exp01_flashing_LEDs.sch (KiCad schematic (older format))
At the start: 248 parts

Commit message: annotating components
Parts:
- gave numbers to parts that had none: 246
Connections:
- net GND: now also SW5.3 (A), SW6.3 (A); no longer SW5.1 (A), SW6.1 (A)
- net at R41.2, R42.2, R43.2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: now also SW5.4 (B), SW6.4 (B); no longer SW5.2 (B), SW6.2 (B)
