File: experiments/schematics/LED_Debug_Board.sch (KiCad schematic (older format))
At the start: 65 parts

Commit message: adding very old modifications
Changed lines of the file:
@@
 	10050 950  10250 950
 Wire Wire Line
-	10250 950  10250 1300
-Wire Wire Line
-	10250 1300 10250 1650
-Wire Wire Line
-	10250 1650 10250 2000
-Wire Wire Line
-	10250 2000 10250 2350
-Wire Wire Line
-	10250 2350 10250 2700
-Wire Wire Line
-	10250 2700 10250 3050
-Wire Wire Line
-	10250 3050 10250 3300
-Wire Wire Line
-	10250 3300 10250 3400
-Wire Wire Line
-	10250 3400 10250 3750
-Wire Wire Line
-	10250 3750 10250 4100
-Wire Wire Line
-	10250 4100 10250 4450
-Wire Wire Line
-	10250 4450 10250 4800
-Wire Wire Line
-	10250 4800 10250 5150
-Wire Wire Line
-	10250 5150 10250 5500
-Wire Wire Line
-	10250 5500 10250 5850
-Wire Wire Line
-	10250 5850 10250 6200
+	10250 950  10250 6200
 Wire Wire Line
 	10250 6200 10050 6200
@@
 $EndComp
 Wire Wire Line
-	10250 1300 10250 1650
-Wire Wire Line
-	10250 1650 10250 2000
-Wire Wire Line
-	10250 2000 10250 2350
-Wire Wire Line
-	10250 2350 10250 2700
-Wire Wire Line
-	10250 2700 10250 3050
-Wire Wire Line
-	10250 3050 10250 3300
-Wire Wire Line
-	10250 3300 10250 3400
-Wire Wire Line
-	10250 3400 10250 3750
-Wire Wire Line
-	10250 3750 10250 4100
-Wire Wire Line
-	10250 4100 10250 4450
-Wire Wire Line
-	10250 4450 10250 4800
-Wire Wire Line
-	10250 4800 10250 5150
-Wire Wire Line
-	10250 5150 10250 5500
-Wire Wire Line
-	10250 5500 10250 5850
+	10250 1300 10250 5850
 $Comp
 L R R?
@@
 $EndComp
 Wire Wire Line
-	10250 1650 10250 2000
-Wire Wire Line
-	10250 2000 10250 2350
-Wire Wire Line
-	10250 2350 10250 2700
-Wire Wire Line
-	10250 2700 10250 3050
-Wire Wire Line
-	10250 3050 10250 3300
-Wire Wire Line
-	10250 3300 10250 3400
-Wire Wire Line
-	10250 3400 10250 3750
-Wire Wire Line
-	10250 3750 10250 4100
-Wire Wire Line
-	10250 4100 10250 4450
-Wire Wire Line
-	10250 4450 10250 4800
-Wire Wire Line
-	10250 4800 10250 5150
-Wire Wire Line
-	10250 5150 10250 5500
+	10250 1650 10250 5500
 $Comp
 L LED_ALT D?
@@
 $EndComp
 Wire Wire Line
-	10250 2000 10250 2350
-Wire Wire Line
-	10250 2350 10250 2700
-Wire Wire Line
-	10250 2700 10250 3050
-Wire Wire Line
-	10250 3050 10250 3300
-Wire Wire Line
-	10250 3300 10250 3400
-Wire Wire Line
-	10250 3400 10250 3750
-Wire Wire Line
-	10250 3750 10250 4100
-Wire Wire Line
-	10250 4100 10250 4450
-Wire Wire Line
-	10250 4450 10250 4800
-Wire Wire Line
-	10250 4800 10250 5150
+	10250 2000 10250 5150
 $Comp
 L CONN_01X40 P?
@@
 Connection ~ 7850 2300
 Wire Wire Line
-	7650 1950 7850 1950
-Wire Wire Line
-	7850 1950 8150 1950
+	7650 1950 8150 1950
 Connection ~ 7850 1950
 Wire Wire Line
@@
 	10250 3300 10550 3300
 Wire Wire Line
-	7850 900  7850 1250
-Wire Wire Line
-	7850 1250 7850 1600
-Wire Wire Line
-	7850 1600 7850 1950
-Wire Wire Line
-	7850 1950 7850 2300
-Wire Wire Line
-	7850 2300 7850 2650
-Wire Wire Line
-	7850 2650 7850 3000
-Wire Wire Line
-	7850 3000 7850 3350
+	7850 900  7850 3350
 $Comp
 L Earth #PWR?
@@
 Connection ~ 7850 5100
 Wire Wire Line
-	7650 4750 7850 4750
-Wire Wire Line
-	7850 4750 8150 4750
+	7650 4750 8150 4750
 Connection ~ 7850 4750
 Wire Wire Line
@@
 	6950 6150 6850 6150
 Wire Wire Line
-	7850 3700 7850 4050
-Wire Wire Line
-	7850 4050 7850 4400
-Wire Wire Line
-	7850 4400 7850 4750
-Wire Wire Line
-	7850 4750 7850 5100
-Wire Wire Line
-	7850 5100 7850 5450
-Wire Wire Line
-	7850 5450 7850 5800
-Wire Wire Line
-	7850 5800 7850 6150
+	7850 3700 7850 6150
 $Comp
 L Earth #PWR?
